File: Rev 2/Buck V1.brd (EAGLE design)
At the start: 160 x 100 mm, 11 parts, among them U1 Value

Commit message: added schematic for Current Driver V2!
Parts:
- added C_COMP1: 1.2 nF, rcl:C0603
- added C_COMP2: 82 pF, rcl:C0603
- added C_IN1, C_IN2, C_IN3, C_IN4: 10 uF, rcl:C1206
- added C_INS1, C_SS: 100 nF, rcl:C0603
- added C_RES: 1 uF, rcl:C0603
- added D_IN: IN4148, adafruit:SOD-123
- added Q1, Q2, Q3, Q4: IRF3205STRLPBF, mixed_components:D2PAK
- added R_COMP: 28.7 K, rcl:R0603
- added R_DIS1, R_UV1: 3.3 K, rcl:R0603
- added R_DIS2, R_UV2: 56 K, rcl:R0603
- added R_FB, R_SHTDWN, R_VOUT1: 1 K, rcl:R0603
- added R_T: 12.1 K, rcl:R0603
- added R_VOUT2: 5 K, rcl:R0603
- renumbered CBOOT to C_BOOT, COUT to C_OUT, COUTS1 to C_OUTS1, COUTS2 to C_OUTS2, CRAMP to C_RAMP, CVCC to C_VCC, DBOOT to D_BOOT, RRAMP to R_RAMP, RSENSE to R_SENSE
Connections:
- removed net AGND: U1.6
- removed net PGND: U1.14
- removed net VIN: U1.20
- new net ARD_CURRENT: U1.10
- new net ARD_FEEDBACK: R_FB.1
- new net ARD_SHUTDOWN: R_SHTDWN.1
- new net ARD_VOUT: R_VOUT1.2, R_VOUT2.1
- new net N$10: D_IN.C, U1.20
- new net N$11: R_SHTDWN.2, R_UV1.1, R_UV2.1, U1.1
- new net N$12: C_IN1.1, C_IN2.1, C_IN3.1, C_IN4.1, C_INS1.1, D_IN.A, Q1.2, Q4.2, R_DIS2.2, R_UV2.2
- new net N$13: R_DIS1.1, R_DIS2.1, U1.7
- new net N$14: C_COMP1.1, C_COMP2.1, U1.9
- new net N$15: C_COMP2.2, R_COMP.1, R_FB.2, U1.8
- new net N$16: R_T.2, U1.5
- new net N$17: C_RES.1, U1.3
- new net N$18: C_SS.1, U1.4
- new net N$7: Q2.1, Q3.1, U1.15
- new net N$8: Q1.1, Q4.1, U1.18
- new net N$9: C_COMP1.2, R_COMP.2
- net GND: now also C_IN1.2, C_IN2.2, C_IN3.2, C_IN4.2, C_INS1.2, C_RES.2, C_SS.2, R_DIS1.2, R_T.1, R_UV1.2, R_VOUT1.1, U1.14, U1.21, U1.6
- net N$3: now also Q1.3, Q2.2, Q3.2, Q4.3
- net N$4: now also Q2.3, Q3.3
- net N$6: now also R_VOUT2.2

Commit message: Added Board Layout for Buck V1 Module
Parts:
- added C_CURR: 100 pF, rcl:C0603
- added C_VIN: 1 UF, rcl:C0603
- added JP1: (no value), adafruit:1X06
- added R_CURR1, R_CURR2: 100, rcl:R0603
- added TP1, TP10, TP11, TP2, TP3, TP4, TP5, TP6, TP7, TP8, TP9: PTR1TP20R, testpad:TP20R
- C_VCC: value 1 UF 25V -> 1 UF
- U1: value Value -> LM5117
- moved R_VOUT2 233.9 mm to (54.6, 23.2)
- moved R_VOUT1 233.0 mm to (52.1, 19.7), turned to 90 degrees
- moved C_IN4 211.6 mm to (10.8, 25.1), turned to 270 degrees
- moved C_IN3 206.8 mm to (14.6, 25.1), turned to 270 degrees
- moved C_IN2 202.3 mm to (18.4, 25.1), turned to 270 degrees
- moved C_IN1 197.9 mm to (22.2, 25.1), turned to 270 degrees
- moved C_INS1 195.4 mm to (26.0, 25.1), turned to 270 degrees
- moved C_SS 184.1 mm to (40.0, 9.53)
- moved R_FB 180.6 mm to (47.0, 14.6), turned to 180 degrees
- moved C_RES 178.2 mm to (40.0, 7.62)
- moved R_T 177.2 mm to (40.0, 11.4), turned to 180 degrees
- moved R_COMP 174.8 mm to (43.2, 15.2)
- moved C_COMP2 171.0 mm to (40.6, 16.2), turned to 270 degrees
- moved C_COMP1 170.2 mm to (43.2, 17.1)
- moved R_DIS1 161.9 mm to (42.9, 12.1), turned to 270 degrees
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Connections:
- removed net N$12: C_IN1.1, C_IN2.1, C_IN3.1, C_IN4.1, C_INS1.1, D_IN.A, Q1.2, Q4.2, R_DIS2.2, R_UV2.2
- removed net N$6: C_OUT.P$2, C_OUTS1.1, C_OUTS2.1, L1.2, R_VOUT2.2
- new net N$19: C_CURR.1, R_CURR1.1, U1.12
- new net N$20: C_CURR.2, R_CURR2.1, U1.13
- new net N$21: C_IN1.1, C_IN2.1, C_IN3.1, C_IN4.1, C_INS1.1, D_IN.A, Q1.2, Q4.2, R_UV2.2, TP1.TP
- new net V_OUT: C_OUT.P$2, C_OUTS1.1, C_OUTS2.1, L1.2, R_DIS2.2, R_VOUT2.2, TP8.TP
- net ARD_CURRENT: now also JP1.2, TP4.TP
- net ARD_FEEDBACK: now also JP1.3, TP3.TP
- net ARD_SHUTDOWN: now also JP1.1, TP2.TP
- net ARD_VOUT: now also JP1.4, TP6.TP
- net GND: now also C_VIN.2, JP1.5, JP1.6, R_CURR2.2; no longer U1.13
- net N$1: now also TP5.TP
- net N$10: now also C_VIN.1
- net N$3: now also TP7.TP
- net N$4: now also R_CURR1.2, TP11.TP; no longer U1.12
- net N$7: now also TP10.TP
- net N$8: now also TP9.TP
Routing:
- net ARD_VOUT: track 0.00 -> 53.5 mm, vias 0 -> 1
- net N$8: track 0.00 -> 53.0 mm, vias 0 -> 3
- net N$3: track 0.00 -> 44.8 mm, vias 0 -> 95
- net ARD_FEEDBACK: track 0.00 -> 42.2 mm, vias 0 -> 1
- net ARD_CURRENT: track 0.00 -> 39.8 mm, vias 0 -> 1
- net N$21: track 0.00 -> 37.9 mm, vias 0 -> 95
- net N$7: track 0.00 -> 36.0 mm, vias 0 -> 3
- net ARD_SHUTDOWN: track 0.00 -> 29.5 mm, vias 0 -> 1
- net N$4: track 0.00 -> 25.1 mm, vias 0 -> 24
- net N$1: track 0.00 -> 18.4 mm, vias 0 -> 2
- net V_OUT: track 0.00 -> 17.4 mm, vias 0 -> 65
- net N$15: track 0.00 -> 12.1 mm
- net N$13: track 0.00 -> 10.3 mm
- net N$11: track 0.00 -> 9.31 mm
- net N$14: track 0.00 -> 7.45 mm
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- added copper zone on layer 1, net GND
- added copper zone on layer 15, net GND
- added copper zone on layer 16, net GND
- added copper zone on layer 2, net GND
- added copper zone on layer 1, net N$21
- added copper zone on layer 16, net N$21
- added copper zone on layer 1, net N$3
- added copper zone on layer 16, net N$3
- added copper zone on layer 1, net N$4
- added copper zone on layer 16, net N$4
- added copper zone on layer 1, net V_OUT
- added copper zone on layer 16, net V_OUT
Other:
- board size 160 x 100 mm -> 77.5 x 51.1 mm

Commit message: Added test points, arranged silkscreen text
Parts:
- removed TP1, TP10, TP11, TP2, TP3, TP4, TP5, TP6, TP7, TP8, TP9: PTR1TP20R, testpad:TP20R
- added ARD_CURR, ARD_FB, ARD_SHTDWN, ARD_VOUT, CURR_SENSE, HO, LO, SW, VCC, V_IN, V_OUT: PTR1TP20R, testpad:TP20R
- U1: value LM5117 -> Value
Connections:
- net ARD_CURRENT: now also ARD_CURR.TP; no longer TP4.TP
- net ARD_FEEDBACK: now also ARD_FB.TP; no longer TP3.TP
- net ARD_SHUTDOWN: now also ARD_SHTDWN.TP; no longer TP2.TP
- net ARD_VOUT: now also ARD_VOUT.TP; no longer TP6.TP
- net N$1: now also VCC.TP; no longer TP5.TP
- net N$21: now also V_IN.TP; no longer TP1.TP
- net N$3: now also SW.TP; no longer TP7.TP
- net N$4: now also CURR_SENSE.TP; no longer TP11.TP
- net N$7: now also LO.TP; no longer TP10.TP
- net N$8: now also HO.TP; no longer TP9.TP
- net V_OUT: now also V_OUT.TP; no longer TP8.TP
Routing:
- net N$4: track 25.1 -> 30.3 mm, vias 24 -> 22
- net V_OUT: track 17.4 -> 20.4 mm
- net N$1: track 18.4 -> 21.0 mm
- net ARD_SHUTDOWN: track 29.5 -> 32.1 mm
- net ARD_VOUT: track 53.5 -> 56.0 mm
- net ARD_FEEDBACK: track 42.2 -> 44.7 mm
- net ARD_CURRENT: track 39.8 -> 42.4 mm
- net N$7: track 36.0 -> 38.2 mm
- net N$8: track 53.0 -> 55.3 mm
