File: Rev 2/Buck V1.sch (EAGLE design)
At the start: 11 parts, among them U1 Value

Commit message: added schematic for Current Driver V2!
Parts:
- removed CBOOT: 470 nF 50V, rcl:C-USC0603
- removed COUT: 470 uF, custom-parts:CAP_PANASONIC_H13
- removed COUTS1, COUTS2: 1 uF, rcl:C-USC0805
- removed CRAMP: 820pF 50V, rcl:C-USC0603
- removed RRAMP: 180 KOhm, rcl:R-US_R0603
- removed RSENSE: 1W 5mOhm, rcl:R-US_R2512
- added C_BOOT: 470 nF 50V, rcl:C-USC0603
- added C_COMP1: 1.2 nF, rcl:C-USC0603
- added C_COMP2: 82 pF, rcl:C-USC0603
- added C_IN1, C_IN2, C_IN3, C_IN4: 10 uF, rcl:C-USC1206
- added C_INS1, C_SS: 100 nF, rcl:C-USC0603
- added C_OUT: 470 uF, custom-parts:CAP_PANASONIC_H13
- added C_OUTS1, C_OUTS2: 1 uF, rcl:C-USC0805
- added C_RAMP: 820pF 50V, rcl:C-USC0603
- added C_RES: 1 uF, rcl:C-USC0603
- added D_IN: IN4148, adafruit:DIODESOD-123
- added Q1, Q2, Q3, Q4: IRF3205STRLPBF, mixed_components:IRF510D2PAK
- added R_COMP: 28.7 K, rcl:R-US_R0603
- added R_DIS1, R_UV1: 3.3 K, rcl:R-US_R0603
- added R_DIS2, R_UV2: 56 K, rcl:R-US_R0603
- added R_FB, R_SHTDWN, R_VOUT1: 1 K, rcl:R-US_R0603
- added R_RAMP: 180 KOhm, rcl:R-US_R0603
- added R_SENSE: 1W 5mOhm, rcl:R-US_R2512
- added R_T: 12.1 K, rcl:R-US_R0603
- added R_VOUT2: 5 K, rcl:R-US_R0603
- renumbered CVCC to C_VCC, DBOOT to D_BOOT
Connections:
- new net ARD_CURRENT: U1.CM
- new net ARD_FEEDBACK: R_FB.1
- new net ARD_SHUTDOWN: R_SHTDWN.1
- new net ARD_VOUT: R_VOUT1.2, R_VOUT2.1
- new net N$10: D_IN.C, U1.VIN
- new net N$11: R_SHTDWN.2, R_UV1.1, R_UV2.1, U1.UVLO
- new net N$12: C_IN1.1, C_IN2.1, C_IN3.1, C_IN4.1, C_INS1.1, D_IN.A, Q1.D, Q4.D, R_DIS2.2, R_UV2.2
- new net N$13: R_DIS1.1, R_DIS2.1, U1.VCCDIS
- new net N$14: C_COMP1.1, C_COMP2.1, U1.COMP
- new net N$15: C_COMP2.2, R_COMP.1, R_FB.2, U1.FB
- new net N$16: R_T.2, U1.RT
- new net N$17: C_RES.1, U1.RES
- new net N$18: C_SS.1, U1.SS
- new net N$7: Q2.G, Q3.G, U1.LO
- new net N$8: Q1.G, Q4.G, U1.HO
- new net N$9: C_COMP1.2, R_COMP.2
- net GND: now also C_IN1.2, C_IN2.2, C_IN3.2, C_IN4.2, C_INS1.2, C_OUT.1, C_OUTS1.2, C_OUTS2.2, C_RAMP.2, C_RES.2, C_SS.2, R_DIS1.2, R_SENSE.2, R_T.1, R_UV1.2, R_VOUT1.1, U1.AGND, U1.EP, U1.PGND; no longer COUT.1, COUTS1.2, COUTS2.2, CRAMP.2, RSENSE.2
- net N$2: now also C_BOOT.1; no longer CBOOT.1
- net N$3: now also C_BOOT.2, Q1.S, Q2.D, Q3.D, Q4.S, R_RAMP.2; no longer CBOOT.2, RRAMP.2
- net N$4: now also Q2.S, Q3.S, R_SENSE.1; no longer RSENSE.1
- net N$5: now also C_RAMP.1, R_RAMP.1; no longer CRAMP.1, RRAMP.1
- net N$6: now also C_OUT.2, C_OUTS1.1, C_OUTS2.1, R_VOUT2.2; no longer COUT.2, COUTS1.1, COUTS2.1
Other:
- moved on the sheet: L1

Commit message: Added Board Layout for Buck V1 Module
Parts:
- added C_CURR: 100 pF, rcl:C-USC0603
- added C_VIN: 1 UF, rcl:C-USC0603
- added JP1: (no value), adafruit:PINHD-1X6
- added R_CURR1, R_CURR2: 100, rcl:R-US_R0603
- added TP1, TP10, TP11, TP2, TP3, TP4, TP5, TP6, TP7, TP8, TP9: PTR1TP20R, testpad:PTR1TP20R
- C_IN4: SPICEPREFIX (none) -> C
- C_VCC: value 1 UF 25V -> 1 UF
- U1: value Value -> LM5117
Connections:
- removed net N$12: C_IN1.1, C_IN2.1, C_IN3.1, C_IN4.1, C_INS1.1, D_IN.A, Q1.D, Q4.D, R_DIS2.2, R_UV2.2
- removed net N$6: C_OUT.2, C_OUTS1.1, C_OUTS2.1, L1.2, R_VOUT2.2
- new net N$19: C_CURR.1, R_CURR1.1, U1.CS
- new net N$20: C_CURR.2, R_CURR2.1, U1.CSG
- new net N$21: C_IN1.1, C_IN2.1, C_IN3.1, C_IN4.1, C_INS1.1, D_IN.A, Q1.D, Q4.D, R_UV2.2, TP1.TP
- new net V_OUT: C_OUT.2, C_OUTS1.1, C_OUTS2.1, L1.2, R_DIS2.2, R_VOUT2.2, TP8.TP
- net ARD_CURRENT: now also JP1.2, TP4.TP
- net ARD_FEEDBACK: now also JP1.3, TP3.TP
- net ARD_SHUTDOWN: now also JP1.1, TP2.TP
- net ARD_VOUT: now also JP1.4, TP6.TP
- net GND: now also C_VIN.2, JP1.5, JP1.6, R_CURR2.2; no longer U1.CSG
- net N$1: now also TP5.TP
- net N$10: now also C_VIN.1
- net N$3: now also TP7.TP
- net N$4: now also R_CURR1.2, TP11.TP; no longer U1.CS
- net N$7: now also TP10.TP
- net N$8: now also TP9.TP
Other:
- moved on the sheet: D_IN

Commit message: Added test points, arranged silkscreen text
Parts:
- U1: value LM5117 -> Value
- renumbered TP1 to V_IN, TP10 to LO, TP11 to CURR_SENSE, TP2 to ARD_SHTDWN, TP3 to ARD_FB, TP4 to ARD_CURR, TP5 to VCC, TP6 to ARD_VOUT, TP7 to SW, TP8 to V_OUT, TP9 to HO
Changed lines of the file:
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@@
 </classes>
 <parts>
-<part name="U1" library="AcceleratedDesigns_Lib" deviceset="LM5117PMHX/NOPB" device="" value="LM5117"/>
+<part name="U1" library="AcceleratedDesigns_Lib" deviceset="LM5117PMHX/NOPB" device="" value="Value"/>
 <part name="D_BOOT" library="diode" library_urn="urn:adsk.eagle:library:210" deviceset="DIODE-" device="SOD123" package3d_urn="urn:adsk.eagle:package:43420/1" value="PMEG10010ELRX"/>
 <part name="C_VCC" library="rcl" library_urn="urn:adsk.eagle:library:334" deviceset="C-US" device="C0603" package3d_urn="urn:adsk.eagle:package:23616/2" value="1 UF"/>
@@
 <part name="SUPPLY13" library="supply2" deviceset="GND" device=""/>
 <part name="JP1" library="adafruit" deviceset="PINHD-1X6" device=""/>
-<part name="TP1" library="testpad" deviceset="PTR1" device="TP20R"/>
-<part name="TP2" library="testpad" deviceset="PTR1" device="TP20R"/>
-<part name="TP3" library="testpad" deviceset="PTR1" device="TP20R"/>
-<part name="TP4" library="testpad" deviceset="PTR1" device="TP20R"/>
-<part name="TP5" library="testpad" deviceset="PTR1" device="TP20R"/>
-<part name="TP6" library="testpad" deviceset="PTR1" device="TP20R"/>
-<part name="TP7" library="testpad" deviceset="PTR1" device="TP20R"/>
-<part name="TP8" library="testpad" deviceset="PTR1" device="TP20R"/>
-<part name="TP9" library="testpad" deviceset="PTR1" device="TP20R"/>
-<part name="TP10" library="testpad" deviceset="PTR1" device="TP20R"/>
-<part name="TP11" library="testpad" deviceset="PTR1" device="TP20R"/>
+<part name="V_IN" library="testpad" deviceset="PTR1" device="TP20R"/>
+<part name="ARD_SHTDWN" library="testpad" deviceset="PTR1" device="TP20R"/>
+<part name="ARD_FB" library="testpad" deviceset="PTR1" device="TP20R"/>
+<part name="ARD_CURR" library="testpad" deviceset="PTR1" device="TP20R"/>
+<part name="VCC" library="testpad" deviceset="PTR1" device="TP20R"/>
+<part name="ARD_VOUT" library="testpad" deviceset="PTR1" device="TP20R"/>
+<part name="SW" library="testpad" deviceset="PTR1" device="TP20R"/>
+<part name="V_OUT" library="testpad" deviceset="PTR1" device="TP20R"/>
+<part name="HO" library="testpad" deviceset="PTR1" device="TP20R"/>
+<part name="LO" library="testpad" deviceset="PTR1" device="TP20R"/>
+<part name="CURR_SENSE" library="testpad" deviceset="PTR1" device="TP20R"/>
 </parts>
 <sheets>
@@
 <attribute name="VALUE" x="306.07" y="93.98" size="1.778" layer="96"/>
 </instance>
-<instance part="TP1" gate="G$1" x="-35.56" y="111.76" smashed="yes">
+<instance part="V_IN" gate="G$1" x="-35.56" y="111.76" smashed="yes">
 <attribute name="NAME" x="-36.576" y="105.41" size="1.778" layer="95" rot="R90"/>
 <attribute name="TP_SIGNAL_NAME" x="-34.29" y="109.22" size="1.778" layer="97"/>
 </instance>
-<instance part="TP2" gate="G$1" x="-63.5" y="86.36" smashed="yes">
+<instance part="ARD_SHTDWN" gate="G$1" x="-63.5" y="86.36" smashed="yes">
 <attribute name="NAME" x="-64.516" y="80.01" size="1.778" layer="95" rot="R90"/>
 <attribute name="TP_SIGNAL_NAME" x="-62.23" y="83.82" size="1.778" layer="97"/>
 </instance>
-<instance part="TP3" gate="G$1" x="-71.12" y="48.26" smashed="yes">
+<instance part="ARD_FB" gate="G$1" x="-71.12" y="48.26" smashed="yes">
 <attribute name="NAME" x="-72.136" y="41.91" size="1.778" layer="95" rot="R90"/>
 <attribute name="TP_SIGNAL_NAME" x="-69.85" y="45.72" size="1.778" layer="97"/>
 </instance>
-<instance part="TP4" gate="G$1" x="-71.12" y="35.56" smashed="yes">
+<instance part="ARD_CURR" gate="G$1" x="-71.12" y="35.56" smashed="yes">
 <attribute name="NAME" x="-72.136" y="29.21" size="1.778" layer="95" rot="R90"/>
 <attribute name="TP_SIGNAL_NAME" x="-69.85" y="33.02" size="1.778" layer="97"/>
 </instance>
-<instance part="TP5" gate="G$1" x="147.32" y="76.2" smashed="yes">
+<instance part="VCC" gate="G$1" x="147.32" y="76.2" smashed="yes">
 <attribute name="NAME" x="146.304" y="69.85" size="1.778" layer="95" rot="R90"/>
 <attribute name="TP_SIGNAL_NAME" x="148.59" y="73.66" size="1.778" layer="97"/>
 </instance>
-<instance part="TP6" gate="G$1" x="292.1" y="22.86" smashed="yes">
+<instance part="ARD_VOUT" gate="G$1" x="292.1" y="22.86" smashed="yes">
 <attribute name="NAME" x="291.084" y="16.51" size="1.778" layer="95" rot="R90"/>
 <attribute name="TP_SIGNAL_NAME" x="293.37" y="20.32" size="1.778" layer="97"/>
 </instance>
-<instance part="TP7" gate="G$1" x="236.22" y="50.8" smashed="yes">
+<instance part="SW" gate="G$1" x="236.22" y="50.8" smashed="yes">
 <attribute name="NAME" x="235.204" y="44.45" size="1.778" layer="95" rot="R90"/>
 <attribute name="TP_SIGNAL_NAME" x="237.49" y="48.26" size="1.778" layer="97"/>
 </instance>
-<instance part="TP8" gate="G$1" x="269.24" y="50.8" smashed="yes">
+<instance part="V_OUT" gate="G$1" x="269.24" y="50.8" smashed="yes">
 <attribute name="NAME" x="268.224" y="44.45" size="1.778" layer="95" rot="R90"/>
 <attribute name="TP_SIGNAL_NAME" x="270.51" y="48.26" size="1.778" layer="97"/>
 </instance>
-<instance part="TP9" gate="G$1" x="200.66" y="66.04" smashed="yes">
+<instance part="HO" gate="G$1" x="200.66" y="66.04" smashed="yes">
 <attribute name="NAME" x="199.644" y="59.69" size="1.778" layer="95" rot="R90"/>
 <attribute name="TP_SIGNAL_NAME" x="201.93" y="63.5" size="1.778" layer="97"/>
 </instance>
-<instance part="TP10" gate="G$1" x="200.66" y="48.26" smashed="yes">
+<instance part="LO" gate="G$1" x="200.66" y="48.26" smashed="yes">
 <attribute name="NAME" x="199.644" y="41.91" size="1.778" layer="95" rot="R90"/>
 <attribute name="TP_SIGNAL_NAME" x="201.93" y="45.72" size="1.778" layer="97"/>
 </instance>
-<instance part="TP11" gate="G$1" x="190.5" y="35.56" smashed="yes">
+<instance part="CURR_SENSE" gate="G$1" x="190.5" y="35.56" smashed="yes">
 <attribute name="NAME" x="189.484" y="29.21" size="1.778" layer="95" rot="R90"/>
 <attribute name="TP_SIGNAL_NAME" x="191.77" y="33.02" size="1.778" layer="97"/>
@@
 <wire x1="137.16" y1="78.74" x2="147.32" y2="78.74" width="0.1524" layer="91"/>
 <junction x="137.16" y="78.74"/>
-<pinref part="TP5" gate="G$1" pin="TP"/>
+<pinref part="VCC" gate="G$1" pin="TP"/>
 <wire x1="147.32" y1="78.74" x2="152.4" y2="78.74" width="0.1524" layer="91"/>
 <junction x="147.32" y="78.74"/>
@@
 <pinref part="Q4" gate="G$1" pin="S"/>
 <wire x1="220.98" y1="58.42" x2="220.98" y2="53.34" width="0.1524" layer="91"/>
-<pinref part="TP7" gate="G$1" pin="TP"/>
+<pinref part="SW" gate="G$1" pin="TP"/>
 <junction x="236.22" y="53.34"/>
 </segment>
@@
 <wire x1="154.94" y1="38.1" x2="190.5" y2="38.1" width="0.1524" layer="91"/>
 <junction x="190.5" y="38.1"/>
-<pinref part="TP11" gate="G$1" pin="TP"/>
+<pinref part="CURR_SENSE" gate="G$1" pin="TP"/>
 </segment>
 </net>
@@
 <junction x="307.34" y="53.34"/>
 <label x="322.58" y="53.34" size="1.778" layer="95"/>
-<pinref part="TP8" gate="G$1" pin="TP"/>
+<pinref part="V_OUT" gate="G$1" pin="TP"/>
 <junction x="269.24" y="53.34"/>
 </segment>
@@
 <pinref part="Q3" gate="G$1" pin="G"/>
 <wire x1="203.2" y1="43.18" x2="210.82" y2="43.18" width="0.1524" layer="91"/>
-<pinref part="TP10" gate="G$1" pin="TP"/>
+<pinref part="LO" gate="G$1" pin="TP"/>
 <junction x="200.66" y="50.8"/>
 </segment>
@@
 <pinref part="Q4" gate="G$1" pin="G"/>
 <wire x1="203.2" y1="58.42" x2="210.82" y2="58.42" width="0.1524" layer="91"/>
-<pinref part="TP9" gate="G$1" pin="TP"/>
+<pinref part="HO" gate="G$1" pin="TP"/>
 <junction x="200.66" y="68.58"/>
 </segment>
@@
 <wire x1="-35.56" y1="88.9" x2="-63.5" y2="88.9" width="0.1524" layer="91"/>
 <label x="-91.44" y="88.9" size="1.778" layer="95"/>
-<pinref part="TP2" gate="G$1" pin="TP"/>
+<pinref part="ARD_SHTDWN" gate="G$1" pin="TP"/>
 <wire x1="-63.5" y1="88.9" x2="-73.66" y2="88.9" width="0.1524" layer="91"/>
 <junction x="-63.5" y="88.9"/>
@@
 <wire x1="-71.12" y1="50.8" x2="-73.66" y2="50.8" width="0.1524" layer="91"/>
 <label x="-91.44" y="50.8" size="1.778" layer="95"/>
-<pinref part="TP3" gate="G$1" pin="TP"/>
+<pinref part="ARD_FB" gate="G$1" pin="TP"/>
 <junction x="-71.12" y="50.8"/>
 </segment>
@@
 <wire x1="-12.7" y1="38.1" x2="-71.12" y2="38.1" width="0.1524" layer="91"/>
 <label x="-91.44" y="38.1" size="1.778" layer="95"/>
-<pinref part="TP4" gate="G$1" pin="TP"/>
+<pinref part="ARD_CURR" gate="G$1" pin="TP"/>
 <wire x1="-71.12" y1="38.1" x2="-73.66" y2="38.1" width="0.1524" layer="91"/>
 <junction x="-71.12" y="38.1"/>
@@
 <wire x1="271.78" y1="25.4" x2="292.1" y2="25.4" width="0.1524" layer="91"/>
 <label x="307.34" y="25.4" size="1.778" layer="95"/>
-<pinref part="TP6" gate="G$1" pin="TP"/>
+<pinref part="ARD_VOUT" gate="G$1" pin="TP"/>
 <wire x1="292.1" y1="25.4" x2="307.34" y2="25.4" width="0.1524" layer="91"/>
 <junction x="292.1" y="25.4"/>
@@
 <junction x="220.98" y="73.66"/>
 <junction x="22.86" y="114.3"/>
-<pinref part="TP1" gate="G$1" pin="TP"/>
+<pinref part="V_IN" gate="G$1" pin="TP"/>
 <junction x="-35.56" y="114.3"/>
 </segment>
